File: PCB/ClonadorDeSeñalesEsp32/ClonadorDeSeñalesEsp32.kicad_pcb (KiCad board)
At the start: 2 copper layers, 100 x 100 mm, 16 parts

Commit message: Fin de la PCB
PCB después de revisión del profesor
Parts:
- moved Servo2 4.50 mm to (89.4, 54.0)
Routing:
- net GND: track 8.00 -> 0.00 mm, vias 2 -> 0
- net +5V: track 212.0 -> 204.6 mm, vias 0 -> 2
- net /servo_2: track 37.6 -> 38.6 mm
- net /resistencia2: track 36.4 -> 36.2 mm, vias 2 -> 0
- net /resistencia1: vias 2 -> 0
Changed lines of the file:
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@@
 	(footprint "Connector_PinHeader_2.54mm:PinHeader_1x03_P2.54mm_Vertical"
 		(layer "F.Cu")
-		(at 89.46 58.5 90)
+		(at 89.42 54 90)
 		(descr "Through hole straight pin header, 1x03, 2.54mm pitch, single row")
 		(tags "Through hole pin header THT 1x03 2.54mm single row")
@@
 	)
 	(segment
-		(start 86.5 58.5)
-		(end 86.5 66.5)
-		(width 0.6)
-		(layer "F.Cu")
-		(net 2)
-	)
-	(via
-		(at 86.5 58.5)
-		(size 1.1)
-		(drill 0.65)
-		(layers "F.Cu" "B.Cu")
-		(net 2)
-	)
-	(via
-		(at 86.5 66.5)
-		(size 1.1)
-		(drill 0.65)
-		(layers "F.Cu" "B.Cu")
-		(net 2)
-	)
-	(segment
 		(start 105 53)
 		(end 105 77.555)
@@
 	)
 	(segment
-		(start 103.515 95.015)
-		(end 106 97.5)
+		(start 145 104)
+		(end 149 104)
 		(width 1)
-		(layer "B.Cu")
+		(layer "F.Cu")
 		(net 4)
 	)
 	(segment
-		(start 93.77 112.23)
-		(end 89.04 112.23)
+		(start 139.5 109.5)
+		(end 145 104)
 		(width 1)
-		(layer "B.Cu")
+		(layer "F.Cu")
 		(net 4)
 	)
 	(segment
-		(start 97 88.5)
-		(end 103.515 95.015)
+		(start 131.5 109.5)
+		(end 139.5 109.5)
 		(width 1)
-		(layer "B.Cu")
+		(layer "F.Cu")
+		(net 4)
+	)
+	(via
+		(at 149 104)
+		(size 1.3)
+		(drill 0.65)
+		(layers "F.Cu" "B.Cu")
+		(net 4)
+	)
+	(via
+		(at 131.5 109.5)
+		(size 1.3)
+		(drill 0.65)
+		(layers "F.Cu" "B.Cu")
 		(net 4)
 	)
 	(segment
-		(start 105.015 93.515)
-		(end 110.8 93.515)
+		(start 91.42 57.5)
+		(end 81.5 57.5)
 		(width 1)
 		(layer "B.Cu")
@@
 	)
 	(segment
-		(start 163 99.5)
-		(end 166.08 96.42)
+		(start 93.77 112.23)
+		(end 89.04 112.23)
 		(width 1)
 		(layer "B.Cu")
@@
 	)
 	(segment
-		(start 166.08 96.42)
-		(end 166.08 89.3)
+		(start 105.015 93.515)
+		(end 110.8 93.515)
 		(width 1)
 		(layer "B.Cu")
@@
 	)
 	(segment
-		(start 106 109.5)
-		(end 138.5 109.5)
+		(start 78 71)
+		(end 78.5 71.5)
 		(width 1)
 		(layer "B.Cu")
@@
 	)
 	(segment
-		(start 106 97.5)
-		(end 106 109.5)
+		(start 163 99.5)
+		(end 166.08 96.42)
 		(width 1)
 		(layer "B.Cu")
@@
 	)
 	(segment
-		(start 81.5 60.5)
-		(end 81.5 54.5)
+		(start 91.96 56.96)
+		(end 91.42 57.5)
 		(width 1)
 		(layer "B.Cu")
@@
 	)
 	(segment
-		(start 76.5 60.5)
-		(end 76.5 70.5)
+		(start 166.08 96.42)
+		(end 166.08 89.3)
 		(width 1)
 		(layer "B.Cu")
@@
 	)
 	(segment
-		(start 97 72.5)
-		(end 97 88.5)
+		(start 131.5 109.5)
+		(end 106 109.5)
 		(width 1)
 		(layer "B.Cu")
@@
 	)
 	(segment
-		(start 77.5 71.5)
-		(end 96 71.5)
+		(start 97 88.5)
+		(end 103.515 95.015)
 		(width 1)
 		(layer "B.Cu")
@@
 	)
 	(segment
-		(start 81.5 60.5)
-		(end 76.5 60.5)
+		(start 78.5 60.5)
+		(end 78 61)
 		(width 1)
 		(layer "B.Cu")
@@
 	)
 	(segment
-		(start 144 104)
-		(end 149 104)
+		(start 106 97.5)
+		(end 103.515 95.015)
 		(width 1)
 		(layer "B.Cu")
@@
 	)
 	(segment
-		(start 81.5 54.5)
-		(end 91.96 54.5)
+		(start 97 72.5)
+		(end 97 88.5)
 		(width 1)
 		(layer "B.Cu")
@@
 	)
 	(segment
-		(start 76.5 70.5)
-		(end 77.5 71.5)
+		(start 153.5 99.5)
+		(end 163 99.5)
 		(width 1)
 		(layer "B.Cu")
@@
 	)
 	(segment
-		(start 153.5 99.5)
-		(end 163 99.5)
+		(start 78.5 71.5)
+		(end 96 71.5)
 		(width 1)
 		(layer "B.Cu")
@@
 	)
 	(segment
-		(start 91.96 58.46)
-		(end 92 58.5)
+		(start 92.5 53.96)
+		(end 91.96 54.5)
 		(width 1)
 		(layer "B.Cu")
@@
 	)
 	(segment
-		(start 92.5 47.46)
-		(end 92.04 47)
+		(start 91.96 54.5)
+		(end 91.96 56.96)
 		(width 1)
 		(layer "B.Cu")
@@
 	)
 	(segment
-		(start 92.5 53.96)
-		(end 92.5 47.46)
+		(start 78 61)
+		(end 78 71)
 		(width 1)
 		(layer "B.Cu")
@@
 	)
 	(segment
-		(start 138.5 109.5)
-		(end 144 104)
+		(start 106 109.5)
+		(end 106 97.5)
 		(width 1)
 		(layer "B.Cu")
@@
 	)
 	(segment
-		(start 91.96 54.5)
-		(end 91.96 58.46)
+		(start 81.5 60.5)
+		(end 78.5 60.5)
 		(width 1)
 		(layer "B.Cu")
@@
 	)
 	(segment
-		(start 91.96 54.5)
-		(end 92.5 53.96)
+		(start 93.77 112.23)
+		(end 102 104)
 		(width 1)
 		(layer "B.Cu")
@@
 	)
 	(segment
-		(start 93.77 112.23)
-		(end 102 104)
+		(start 92.5 47.46)
+		(end 92.5 53.96)
 		(width 1)
 		(layer "B.Cu")
@@
 	)
 	(segment
-		(start 102 104)
-		(end 102 96.53)
+		(start 81.5 57.5)
+		(end 81.5 60.5)
 		(width 1)
 		(layer "B.Cu")
@@
 	)
 	(segment
-		(start 94.54 58.5)
-		(end 100.5 58.5)
-		(width 0.6)
+		(start 92.04 47)
+		(end 92.5 47.46)
+		(width 1)
 		(layer "B.Cu")
-		(net 5)
+		(net 4)
 	)
 	(segment
-		(start 102.5 60.5)
+		(start 102 104)
+		(end 102 96.53)
+		(width 1)
+		(layer "B.Cu")
+		(net 4)
+	)
+	(segment
+		(start 110.8 85.895)
 		(end 102.5 77.595)
 		(width 0.6)
@@
 	(segment
 		(start 102.5 77.595)
-		(end 110.8 85.895)
+		(end 102.5 62)
 		(width 0.6)
 		(layer "B.Cu")
@@
 	)
 	(segment
-		(start 100.5 58.5)
-		(end 102.5 60.5)
+		(start 102.5 62)
+		(end 94.5 54)
 		(width 0.6)
 		(layer "B.Cu")
@@
 	)
 	(segment
-		(start 145.5 108.5)
-		(end 143 106)
-		(width 0.6)
-		(layer "F.Cu")
-		(net 33)
-	)
-	(segment
-		(start 143 106)
-		(end 143 99.5)
-		(width 0.6)
-		(layer "F.Cu")
-		(net 33)
-	)
-	(via
-		(at 143 99.5)
-		(size 1.1)
-		(drill 0.65)
-		(layers "F.Cu" "B.Cu")
-		(net 33)
-	)
-	(via
-		(at 145.5 108.5)
-		(size 1.1)
-		(drill 0.65)
-		(layers "F.Cu" "B.Cu")
-		(net 33)
-	)
-	(segment
-		(start 147.5 108.45)
-		(end 145.55 108.45)
+		(start 145.45 108.45)
+		(end 147.5 108.45)
 		(width 0.6)
 		(layer "B.Cu")
@@
 	)
 	(segment
-		(start 145.55 108.45)
-		(end 145.5 108.5)
+		(start 143 106)
+		(end 145.45 108.45)
 		(width 0.6)
 		(layer "B.Cu")
@@
 	)
 	(segment
-		(start 143 84)
-		(end 143 99.5)
+		(start 143 99.5)
+		(end 143 106)
 		(width 0.6)
 		(layer "B.Cu")
@@
 	)
 	(segment
-		(start 139.5 103)
-		(end 139.5 110)
+		(start 143 84)
+		(end 143 99.5)
 		(width 0.6)
-		(layer "F.Cu")
-		(net 34)
+		(locked yes)
+		(layer "B.Cu")
+		(net 33)
 	)
 	(segment
-		(start 139.5 110)
-		(end 142 112.5)
+		(start 143.5 112.5)
+		(end 143 112)
 		(width 0.6)
-		(layer "F.Cu")
-		(net 34)
-	)
-	(via
-		(at 139.5 103)
-		(size 1.1)
-		(drill 0.65)
-		(layers "F.Cu" "B.Cu")
-		(net 34)
-	)
-	(via
-		(at 142 112.5)
-		(size 1.1)
-		(drill 0.65)
-		(layers "F.Cu" "B.Cu")
+		(layer "B.Cu")
 		(net 34)
 	)
 	(segment
-		(start 147.5 112.5)
-		(end 142 112.5)
+		(start 139.5 86)
+		(end 139.5 108.5)
 		(width 0.6)
 		(layer "B.Cu")
@@
 	)
 	(segment
-		(start 139.5 86)
-		(end 139.5 103)
+		(start 147.5 112.5)
+		(end 143.5 112.5)
 		(width 0.6)
 		(layer "B.Cu")
@@
 		(width 0.6)
 		(layer "B.Cu")
+		(net 34)
+	)
+	(segment
+		(start 139.5 108.5)
+		(end 143.5 112.5)
+		(width 0.6)
+		(layer "B.Cu")
